File: CAN BUS.kicad_sch (KiCad schematic)
At the start: 9 parts, among them U3 SN65HVD232DR, U4 ESDCAN24-2BLY

Commit message: finishing+microchecking
Other:
- note added: "*propagation delay resistor"
Changed lines of the file:
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@@
+		)
+	)
+	(text "*propagation \ndelay resistor"
+		(exclude_from_sim no)
+		(at 138.938 73.152 0)
+		(effects
+			(font
+				(size 1.27 1.27)
+			)
 		)
 	)
