File: MCU.kicad_sch (KiCad schematic)
At the start: 15 parts, among them J1 Conn_01x05_Socket, U1 STM32F405RGT6, Y1 8MHz 10ppm

Commit message: ready for review
1. finish routing
2. finish silkscreen adjustment
3. finish DRC and ERC
Parts:
- added R51: 2.2K, Resistor_SMD:R_0603_1608Metric, symbol Device:R_Small
- added SW1: SW_Push, Button_Switch_SMD:SW_Tactile_SPST_NO_Straight_CK_PTS636Sx25SMTRLFS, symbol Switch:SW_Push
Connections:
- net GND: now also R51.1
- net NRST: now also SW1.2
- new net: R51.2, SW1.1

Commit message: finishing+microchecking
Other:
- moved on the sheet: C1, C10, C11, C12, C2, C3, C4, C5, C6, C7, C8, C9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
