File: POWER REGULATOR.kicad_sch (KiCad schematic)
At the start: 12 parts, among them J7 XT60-M, U2 AMS1117-3.3

Commit message: finishing+microchecking
Parts:
- D3: footprint Diode_SMD:D_SOD-323F -> Diode_SMD:D_SOD-323_HandSoldering
Changed lines of the file:
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@@
 			)
 		)
-		(property "Footprint" "Diode_SMD:D_SOD-323F"
+		(property "Footprint" "Diode_SMD:D_SOD-323_HandSoldering"
 			(at 161.29 64.77 0)
 			(effects
