File: VESC V.2.kicad_pcb (KiCad board)
At the start: 4 copper layers, 123 x 68 mm, 149 parts, among them IC1 DRV8302, J1 Conn_01x05_Socket, J2 USB_C_Receptacle_USB2.0_16P, J3 CAN BUS, J4 HALL SENSOR, J5 Conn_01x07_Socket, J6 Conn_01x03_Socket, J7 XT60-M, Q1 IRFS7530TRL7PP, Q2 IRFS7530TRL7PP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

Commit message: add open hardware logo
Parts:
- added REF**: OSHW-Logo_38.1x40mm_SilkScreen, Symbol:OSHW-Logo_38.1x40mm_SilkScreen, F.Cu at (74.0, 94.3)

Commit message: ready for review
1. finish routing
2. finish silkscreen adjustment
3. finish DRC and ERC
Parts:
- removed REF**: OSHW-Logo_38.1x40mm_SilkScreen, Symbol:OSHW-Logo_38.1x40mm_SilkScreen
- added R51: 2.2K, Resistor_SMD:R_0603_1608Metric, F.Cu at (74.8, 54.7)
- added SW1: SW_Push, Button_Switch_SMD:SW_Tactile_SPST_NO_Straight_CK_PTS636Sx25SMTRLFS, F.Cu at (80.7, 54.2)
- moved C41 4.35 mm to (86.5, 42.0)
- moved C42 4.35 mm to (79.1, 42.9)
- moved R19 4.35 mm to (70.9, 45.7)
- moved R20 4.35 mm to (82.8, 49.2)
- moved R30 4.35 mm to (79.1, 44.6)
- moved U3 4.35 mm to (84.6, 45.6)
- moved U4 4.35 mm to (74.6, 45.6)
- moved C43 4.35 mm to (79.1, 48.2)
- moved R29 4.35 mm to (79.1, 46.5)
Connections:
- C21 pad 1: Net-(C21-Pad1) -> V_SUPPLY
- IC1 pad 53: Net-(C21-Pad1) -> V_SUPPLY
- IC1 pad 54: Net-(C21-Pad1) -> V_SUPPLY
Routing:
- net VCC: track 31.3 -> 288.0 mm, vias 0 -> 18
- net NRST: track 4.51 -> 52.0 mm, vias 1 -> 2
- net V_SUPPLY: track 125.8 -> 145.1 mm, vias 74 -> 128
- net /MOSFET DRIVER/H1_VS: track 53.5 -> 36.5 mm, vias 134 -> 133
- net /MOSFET DRIVER/H2_VS: track 50.2 -> 35.7 mm
- net /MOSFET DRIVER/SH2_B: track 44.6 -> 30.4 mm
- net /MOSFET DRIVER/H3_LOW: track 24.9 -> 32.1 mm, vias 0 -> 17
- net GND: track 0.28 -> 7.28 mm, vias 306 -> 385
- net Net-(D6-A2): track 5.96 -> 12.9 mm
- net +5V: track 216.5 -> 223.0 mm, vias 4 -> 5
- net /CAN BUS/CAN_TX: track 16.3 -> 22.3 mm
- net /CAN BUS/CAN_RX: track 20.3 -> 26.2 mm
- net /HALL_FILTER/TEMP_OUT: track 27.1 -> 21.9 mm
- net /CAN BUS/CANL: track 15.0 -> 20.1 mm
- net /MOSFET DRIVER/SH2_A: track 37.4 -> 32.6 mm
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- added copper zone on B.Cu, net /MOSFET DRIVER/HI_LOW
- added copper zone on In2.Cu, net VCC
- removed copper zone on F.Cu, net Net-(C21-Pad1)

Commit message: finishing+microchecking
Parts:
- added REF**: OSHW-Logo_7.5x8mm_SilkScreen, Symbol:OSHW-Logo_7.5x8mm_SilkScreen, F.Cu at (122.3, 44.8)
- D3: footprint Diode_SMD:D_SOD-323F -> Diode_SMD:D_SOD-323_HandSoldering
- moved D3 0.35 mm to (101.2, 48.8)
- moved J7 0.21 mm to (120.8, 35.3)
- moved J5 0.10 mm to (65.3, 68.1)
- moved J6 0.10 mm to (111.5, 95.1)
Routing:
- net VCC: track 288.0 -> 289.9 mm
- net GND: vias 385 -> 383
